File: zeno_board.kicad_sch (KiCad schematic)
At the start: 0 parts

Commit message: feat: more stuff
Parts:
- added C1: 10u, symbol Device:C
- added C2, C3, C4, C5, C6, C8: 100n, symbol Device:C
- added C7, C9: 1u, symbol Device:C
- added FB1: 600R, symbol Device:FerriteBead
- added U1: STM32F401RETx, Package_QFP:LQFP-64_10x10mm_P0.5mm, symbol MCU_ST_STM32F4:STM32F401RETx
Connections:
- new net +3.3V: C1.2, C2.2, C3.2, C4.2, C5.2, C6.2, C9.2, FB1.1, U1.1 (VBAT), U1.19 (VDD), U1.32 (VDD), U1.48 (VDD), U1.64 (VDD)
- new net +3.3VA: C7.2, C8.2, FB1.2, U1.13 (VREF+)
- new net GND: C1.1, C2.1, C3.1, C4.1, C5.1, C6.1, C7.1, C8.1, C9.1, U1.12 (VSSA), U1.18 (VSS), U1.31 (VSS), U1.47 (VSS), U1.63 (VSS)
Other:
- company: (none) -> mufeedcm
- title: (none) -> Zeno  Board
